File: Z88_1MB_Flash/z88-flash-mod.kicad_pcb (KiCad board)
At the start: 4 copper layers, 50.6 x 52.5 mm, 11 parts, among them J1 Conn_Z88, U1 AM29F800B [JEDEC 1024k x8 / 5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, U2 HY628400A LLG-70, U3 HY628400A LLG-70, U4 74LS139

Commit message: minor edits
Parts:
- added QR_code: LOGO, LOGO, B.Cu at (154.6, 71.6)
