File: Z88 Flash KiCad/z88-flash-mod.kicad_pcb (KiCad board)
At the start: 4 copper layers, 50.6 x 52.5 mm, 12 parts, among them J1 Conn_Z88, U1 AM29F800B [JEDEC 1024k x8 / 5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, U2 HY628400A LLG-70, U3 HY628400A LLG-70, U4 74LS139

Commit message: small tweaks to schematic, silkscreen, edge cuts, added PDF plot of schematic
Parts:
- JP1: renamed from 512K; value 512KB RAM -> 512k
Other:
- board size 50.6 x 52.5 mm -> 50.5 x 52.5 mm
Changed lines of the file:
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@@
 		(pad_to_mask_clearance 0)
 		(allow_soldermask_bridges_in_footprints no)
-		(grid_origin 132.969 68.199)
+		(grid_origin 115.697 62.992)
 		(pcbplotparams
 			(layerselection 0x00010fc_ffffffff)
@@
 		(descr "SMD Solder Jumper, 1x1.5mm Pads, 0.3mm gap, open")
 		(tags "solder jumper open")
-		(property "Reference" "512K"
+		(property "Reference" "JP1"
 			(at 0.015 -1.875 90)
-			(layer "F.SilkS")
+			(layer "F.Fab")
 			(effects
 				(font
@@
 			)
 		)
-		(property "Value" "512KB RAM"
+		(property "Value" "512k"
 			(at 0 1.9 90)
-			(layer "F.Fab")
+			(layer "F.SilkS")
 			(effects
 				(font
@@
 		(layer "B.SilkS")
 	)
-	(gr_line
-		(start 116.586 76.2)
-		(end 117.094 76.2)
-		(stroke
-			(width 0.12)
-			(type solid)
-		)
-		(layer "F.SilkS")
-	)
-	(gr_line
-		(start 116.586 76.708)
-		(end 117.094 76.708)
-		(stroke
-			(width 0.12)
-			(type solid)
-		)
-		(layer "F.SilkS")
-	)
-	(gr_line
-		(start 116.586 74.422)
-		(end 116.586 75.692)
-		(stroke
-			(width 0.12)
-			(type solid)
-		)
-		(layer "F.SilkS")
-	)
-	(gr_line
-		(start 116.586 76.454)
-		(end 117.094 76.454)
-		(stroke
-			(width 0.12)
-			(type solid)
-		)
-		(layer "F.SilkS")
-	)
-	(gr_line
-		(start 116.078 74.422)
-		(end 116.586 74.422)
-		(stroke
-			(width 0.12)
-			(type solid)
-		)
-		(layer "F.SilkS")
-	)
-	(gr_line
-		(start 116.586 76.454)
-		(end 116.586 76.708)
-		(stroke
-			(width 0.12)
-			(type solid)
-		)
-		(layer "F.SilkS")
-	)
-	(gr_line
-		(start 117.126 73.279)
-		(end 116.11 74.295)
-		(stroke
-			(width 0.12)
-			(type solid)
-		)
-		(layer "F.SilkS")
-	)
-	(gr_line
-		(start 116.586 75.946)
-		(end 117.094 75.946)
-		(stroke
-			(width 0.12)
-			(type solid)
-		)
-		(layer "F.SilkS")
-	)
-	(gr_line
-		(start 117.094 76.454)
-		(end 116.586 76.454)
-		(stroke
-			(width 0.12)
-			(type solid)
-		)
-		(layer "F.SilkS")
-	)
-	(gr_line
-		(start 116.586 75.946)
-		(end 116.586 76.2)
-		(stroke
-			(width 0.12)
-			(type solid)
-		)
-		(layer "F.SilkS")
-	)
-	(gr_line
-		(start 116.586 75.692)
-		(end 117.094 75.692)
-		(stroke
-			(width 0.12)
-			(type solid)
-		)
-		(layer "F.SilkS")
-	)
-	(gr_line
-		(start 118.11 74.422)
-		(end 117.602 74.422)
-		(stroke
-			(width 0.12)
-			(type solid)
-		)
-		(layer "F.SilkS")
-	)
-	(gr_line
-		(start 117.602 76.2)
-		(end 117.094 76.2)
-		(stroke
-			(width 0.12)
-			(type solid)
-		)
-		(layer "F.SilkS")
-	)
-	(gr_line
-		(start 117.602 75.946)
-		(end 117.094 75.946)
-		(stroke
-			(width 0.12)
-			(type solid)
-		)
-		(layer "F.SilkS")
-	)
-	(gr_line
-		(start 117.602 74.422)
-		(end 117.602 75.692)
-		(stroke
-			(width 0.12)
-			(type solid)
-		)
-		(layer "F.SilkS")
-	)
-	(gr_line
-		(start 117.602 76.454)
-		(end 117.094 76.454)
-		(stroke
-			(width 0.12)
-			(type solid)
-		)
-		(layer "F.SilkS")
-	)
-	(gr_line
-		(start 117.602 75.692)
-		(end 117.094 75.692)
-		(stroke
-			(width 0.12)
-			(type solid)
-		)
-		(layer "F.SilkS")
-	)
-	(gr_line
-		(start 117.126 73.279)
-		(end 118.142 74.295)
-		(stroke
-			(width 0.12)
-			(type solid)
-		)
-		(layer "F.SilkS")
-	)
-	(gr_line
-		(start 117.602 76.708)
-		(end 117.094 76.708)
-		(stroke
-			(width 0.12)
-			(type solid)
-		)
-		(layer "F.SilkS")
-	)
-	(gr_line
-		(start 117.602 76.454)
-		(end 117.602 76.708)
-		(stroke
-			(width 0.12)
-			(type solid)
-		)
-		(layer "F.SilkS")
-	)
-	(gr_line
-		(start 117.602 75.946)
-		(end 117.602 76.2)
-		(stroke
-			(width 0.12)
-			(type solid)
-		)
-		(layer "F.SilkS")
-	)
-	(gr_line
-		(start 166.211 86.741)
-		(end 166.243 63.246)
-		(stroke
-			(width 0.05)
-			(type default)
-		)
-		(layer "Edge.Cuts")
-	)
 	(gr_circle
 		(center 147.828 76.2)
@@
 	)
 	(gr_line
-		(start 115.665 111.141)
-		(end 115.665 86.741)
-		(stroke
-			(width 0.05)
-			(type default)
-		)
-		(layer "Edge.Cuts")
-	)
-	(gr_line
 		(start 115.697 63.246)
 		(end 115.951 62.992)
@@
 	(gr_line
 		(start 120.015 115.459)
-		(end 115.665 111.141)
+		(end 115.697 111.125)
 		(stroke
 			(width 0.05)
@@
 	)
 	(gr_line
-		(start 166.211 111.141)
+		(start 166.243 111.125)
 		(end 161.893 115.459)
 		(stroke
@@
 	)
 	(gr_line
-		(start 166.211 86.741)
-		(end 166.211 111.141)
+		(start 115.697 63.246)
+		(end 115.697 111.125)
 		(stroke
 			(width 0.05)
@@
 	)
 	(gr_line
-		(start 115.665 86.741)
-		(end 115.697 63.246)
+		(start 166.243 63.246)
+		(end 166.243 111.125)
 		(stroke
 			(width 0.05)
